File: Hardware/Main_board.sch (EAGLE design)
At the start: 19 parts, among them IC1 MEGA8-AI, IC2 LP2950CZ-3.0

Commit message: added battery voltage sensing HW
Parts:
- added R6: 50k, resistor:R-EU_M1206
- added R7: 100k, resistor:R-EU_M1206
Connections:
- new net BATT: IC1.PC1(ADC1), R6.1, R7.1
- net GND: now also R7.2
- net V+: now also R6.2
Changed lines of the file:
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@@
 <part name="TP1" library="testpad" deviceset="TP" device="B2,54"/>
 <part name="GND9" library="supply1" deviceset="GND" device=""/>
+<part name="R6" library="resistor" deviceset="R-EU_" device="M1206" value="50k"/>
+<part name="R7" library="resistor" deviceset="R-EU_" device="M1206" value="100k"/>
+<part name="GND10" library="supply1" deviceset="GND" device=""/>
+<part name="P+3" library="supply1" deviceset="V+" device=""/>
 </parts>
 <sheets>
@@
 <instance part="TP1" gate="G$1" x="91.44" y="81.28"/>
 <instance part="GND9" gate="1" x="91.44" y="71.12"/>
+<instance part="R6" gate="G$1" x="38.1" y="25.4" rot="R90"/>
+<instance part="R7" gate="G$1" x="38.1" y="10.16" rot="R270"/>
+<instance part="GND10" gate="1" x="38.1" y="0"/>
+<instance part="P+3" gate="1" x="38.1" y="35.56"/>
 </instances>
 <busses>
@@
 <pinref part="JP2" gate="A" pin="1"/>
 <pinref part="P+2" gate="1" pin="V+"/>
+</segment>
+<segment>
+<pinref part="R6" gate="G$1" pin="2"/>
+<pinref part="P+3" gate="1" pin="V+"/>
+<wire x1="38.1" y1="30.48" x2="38.1" y2="33.02" width="0.1524" layer="91"/>
 </segment>
 </net>
@@
 <pinref part="GND9" gate="1" pin="GND"/>
 </segment>
+<segment>
+<pinref part="GND10" gate="1" pin="GND"/>
+<pinref part="R7" gate="G$1" pin="2"/>
+<wire x1="38.1" y1="2.54" x2="38.1" y2="5.08" width="0.1524" layer="91"/>
+</segment>
 </net>
 <net name="RXTX" class="0">
@@
 </segment>
 </net>
+<net name="BATT" class="0">
+<segment>
+<pinref part="R6" gate="G$1" pin="1"/>
+<pinref part="R7" gate="G$1" pin="1"/>
+<wire x1="38.1" y1="20.32" x2="38.1" y2="17.78" width="0.1524" layer="91"/>
+<wire x1="38.1" y1="17.78" x2="38.1" y2="15.24" width="0.1524" layer="91"/>
+<wire x1="38.1" y1="17.78" x2="48.26" y2="17.78" width="0.1524" layer="91"/>
+<junction x="38.1" y="17.78"/>
+<label x="43.18" y="17.78" size="1.778" layer="95"/>
+</segment>
+<segment>
+<pinref part="IC1" gate="G$1" pin="PC1(ADC1)"/>
+<wire x1="10.16" y1="91.44" x2="22.86" y2="91.44" width="0.1524" layer="91"/>
+<label x="17.78" y="91.44" size="1.778" layer="95"/>
+</segment>
+</net>
